File: PCB/project.kicad_pcb (KiCad board)
At the start: 2 copper layers, 46.2 x 41.8 mm, 29 parts, among them J1 USB_C_Receptacle_USB2.0_16P, J2 Conn_01x15, J3 Conn_01x15, J4 DISPLAY, Q1 SS8050, Q2 SS8050, U1 CH340C, U2 ESP32-WROOM-32, U3 AMS1117-3.3

Commit message: Added v2 project files(.pcb .pro .sch)
Parts:
- removed J3: Conn_01x15, Connector_PinHeader_2.54mm:PinHeader_1x15_P2.54mm_Vertical
- added J5: Conn_01x10, Connector_PinSocket_2.54mm:PinSocket_1x10_P2.54mm_Vertical, F.Cu at (36.3, 60.1)
- J1: footprint Connector_USB:USB_C_Receptacle_HRO_TYPE-C-31-M-12 -> Connector_USB:USB_C_Receptacle_GCT_USB4105-xx-A_16P_TopMnt_Horizontal
- moved REF** 2.00 mm to (27.8, 28.2)
- renumbered RST to SW1, BOOT to SW2
Routing:
- net /3.3V: track 59.1 -> 108.0 mm, vias 0 -> 2
- net /D22: track 4.18 -> 39.5 mm, vias 0 -> 2
- net /D21: track 6.25 -> 27.7 mm, vias 0 -> 1
- net GND: track 289.5 -> 307.6 mm, vias 27 -> 29
- net /D15: track 37.2 -> 23.7 mm, vias 0 -> 2
- net /D4: track 45.2 -> 32.6 mm
- net /D2: track 70.1 -> 58.7 mm, vias 4 -> 3
- net /D5: track 47.7 -> 38.2 mm
- net /D19: track 7.29 -> 16.4 mm, vias 0 -> 2
- net /D18: track 41.1 -> 32.1 mm
- net /RXD2: track 11.5 -> 5.97 mm
- net /TXD: track 33.5 -> 38.6 mm
- net /RXD: track 54.6 -> 50.0 mm
- net /D23: track 48.3 -> 43.9 mm
- net /USB_D+: track 21.3 -> 22.5 mm
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Other:
- board size 46.2 x 41.8 mm -> 48 x 41.9 mm
- board text removed: "X"
