File: PCB/project.kicad_sch (KiCad schematic)
At the start: 27 parts, among them J1 USB_C_Receptacle_USB2.0_16P, J2 Conn_01x15, J3 Conn_01x15, J4 DISPLAY, Q1 SS8050, Q2 SS8050, SW1 SW_Push, SW2 SW_Push, U1 CH340C, U2 ESP32-WROOM-32, U3 AMS1117-3.3

Commit message: Added v2 project files(.pcb .pro .sch)
Parts:
- removed J3: Conn_01x15, Connector_PinHeader_2.54mm:PinHeader_1x15_P2.54mm_Vertical, symbol Connector_Generic:Conn_01x15
- added J5: Conn_01x10, Connector_PinSocket_2.54mm:PinSocket_1x10_P2.54mm_Vertical, symbol Connector_Generic:Conn_01x10
- J1: footprint Connector_USB:USB_C_Receptacle_HRO_TYPE-C-31-M-12 -> Connector_USB:USB_C_Receptacle_GCT_USB4105-xx-A_16P_TopMnt_Horizontal
Connections:
- net 3.3V: now also J5.10 (Pin_10)
- net D15: now also J5.8 (Pin_8)
- net D19: now also J5.5 (Pin_5)
- net D21: now also J5.4 (Pin_4)
- net D22: now also J5.1 (Pin_1)
- net GND: now also J5.9 (Pin_9)
- net RXD: now also J5.3 (Pin_3)
- net RXD2: now also J5.7 (Pin_7)
- net TXD: now also J5.2 (Pin_2)
- net TXD2: now also J5.6 (Pin_6)
